File: libraries/design-blocks/design-block.kicad_blocks/dc-dc-6.8V10A.kicad_block/dc-dc-6.8V10A.kicad_pcb (KiCad board)
At the start: 4 copper layers, 8 parts, among them P1 1.8mm_16AWG, P2 1.8mm_16AWG, P3 1.8mm_16AWG, P4 1.8mm_16AWG

Commit message: update
Parts:
- H5, H6, H7, H8: footprint MountingHole:MountingHole_3.2mm_M3_DIN965_Pad -> bio-robot:MountingHole_3.2mm_M3_DIN965_Pad
- moved P2 58.1 mm to (117.5, 77.7)
- moved P3 53.1 mm to (148.0, 77.7)
- moved P4 49.7 mm to (148.0, 83.7)
- moved H5 49.2 mm to (117.2, 65.2)
- moved H6 49.1 mm to (147.2, 65.2)
- moved H7 49.1 mm to (117.2, 90.2)
- moved H8 49.1 mm to (147.2, 90.2)
- moved P1 46.1 mm to (117.5, 71.7)
