File: servo-board/servo-board.kicad_pcb (KiCad board)
At the start: 2 copper layers, 77 x 62 mm, 17 parts, among them J1 Screw_Terminal_01x02, J2 Screw_Terminal_01x02, J3 Conn_02x10_Counter_Clockwise, M1 Motor_Servo, M2 Motor_Servo, M3 Motor_Servo, M4 Motor_Servo, M5 Motor_Servo, M6 Motor_Servo, M7 Motor_Servo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

Commit message: board done
Parts:
- added C1: 1uF, bio-robot:C_0603_1608Metric, F.Cu at (168.5, 104.0)
- added C2: 1uF, bio-robot:C_0603_1608Metric, F.Cu at (168.0, 110.0)
- added R1: 100k, bio-robot:R_0603_1608Metric, F.Cu at (166.2, 112.8)
- added U3: ADUM1401CRWZ, bio-robot:SOIC-16W_7.5x10.3mm_P1.27mm, F.Cu at (173.6, 115.0)
- added U4: ADUM1401CRWZ, bio-robot:SOIC-16W_7.5x10.3mm_P1.27mm, F.Cu at (134.5, 115.0)
- added U5: LDO_MIC5206-5.0YM5-TR, bots:SOT-23-5, F.Cu at (167.5, 107.0)
- H1, H2, H3, H4: footprint MountingHole:MountingHole_3.2mm_M3_DIN965_Pad -> bio-robot:MountingHole_3.2mm_M3_DIN965_Pad
- J1, J2: footprint TerminalBlock:TerminalBlock_MaiXu_MX126-5.0-02P_1x02_P5.00mm -> bio-robot:TerminalBlock_MaiXu_MX126-5.0-02P_1x02_P5.00mm
- J3: footprint Connector_PinSocket_2.54mm:PinSocket_2x10_P2.54mm_Vertical -> bio-robot:PinSocket_2x10_P2.54mm_Vertical
- M1, M2, M3, M4, M5, M6, M7, M8: footprint Connector_PinSocket_2.54mm:PinSocket_1x03_P2.54mm_Vertical -> bio-robot:PinSocket_1x03_P2.54mm_Vertical
- moved J2 26.4 mm to (175.5, 153.5), turned to 0 degrees
- moved M5 12.8 mm to (124.5, 118.0)
- moved M8 12.8 mm to (124.5, 106.0)
- moved M1 6.46 mm to (185.4, 118.0)
- moved M2 6.46 mm to (185.4, 114.0)
- moved M3 6.46 mm to (185.4, 110.0)
- moved M4 6.46 mm to (185.4, 106.0)
- moved M6 6.04 mm to (124.5, 114.0)
- moved M7 6.04 mm to (124.5, 110.0)
- moved U2 2.00 mm to (155.0, 111.5)
- moved J1 0.75 mm to (129.5, 153.5)
- moved J3 0.08 mm to (165.5, 155.5)
Connections:
- net /GPIO19_USB_D- renamed /USB_D-
- net /GPIO20_USB_D+ renamed /USB_D+
- net /GPIO46 renamed /FLAG
- J3 pad 5: /GPIO3 -> /GPIO14
- M1 pad 1: /PWM_M1 -> /servos/PWM_M1_ISO
- M2 pad 1: /PWM_M2 -> /servos/PWM_M2_ISO
- M3 pad 1: /PWM_M3 -> /servos/PWM_M3_ISO
- M4 pad 1: /PWM_M4 -> /servos/PWM_M4_ISO
- M5 pad 1: /PWM_M5 -> /servos/PWM_M5_ISO
- M6 pad 1: /PWM_M6 -> /servos/PWM_M6_ISO
- M7 pad 1: /PWM_M7 -> /servos/PWM_M7_ISO
- M8 pad 1: /PWM_M8 -> /servos/PWM_M8_ISO
- U1 pad J1_13: /GPIO3 -> /INT
- U1 pad J1_16: /INT -> /PWM_M8
- U1 pad J1_17: /PWM_M5 -> /PWM_M7
- U1 pad J1_19: /PWM_M7 -> /PWM_M5
- U1 pad J1_20: /PWM_M8 -> /GPIO14
Routing:
- net /FLAG: track 0.00 -> 89.5 mm, vias 0 -> 2
- net /GPIO14: track 0.00 -> 67.2 mm, vias 0 -> 1
- net /GPIO15: track 0.00 -> 33.5 mm
- net /GPIO18: track 0.00 -> 33.5 mm
- net /GPIO16: track 0.00 -> 33.5 mm
- net /GPIO17: track 0.00 -> 33.5 mm
- net /INT: track 0.00 -> 19.4 mm, vias 0 -> 1
- net /USB_D+: track 0.00 -> 17.2 mm
- net /USB_D-: track 0.00 -> 16.1 mm
- net +5VA: track 0.00 -> 14.6 mm, vias 0 -> 5
- net GNDPWR: track 0.00 -> 13.8 mm, vias 0 -> 6
- net /SCL: track 0.00 -> 11.9 mm
- net /servos/PWM_M4_ISO: track 0.00 -> 11.6 mm
- net /servos/PWM_M1_ISO: track 0.00 -> 11.2 mm
- net /servos/PWM_M5_ISO: track 0.00 -> 10.3 mm
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- added copper zone on In2.Cu, net +3V3
- added copper zone on F.Cu, net +5V
- added copper zone on In2.Cu, net +5VA
- added copper zone on In2.Cu, net +6.8V
- added copper zone on In1.Cu, net GND
- added copper zone on In1.Cu, net GNDPWR
Other:
- copper layers 2 -> 4
- rule pad_to_mask_clearance: 0 -> 0.1016
- board text added: "5V"
- board text added: "6.8V"
- board text added: "GND"
- board text added: "GNDPWR"
- board text added: "MECH 540 / EECE 571M Marine Robotics Group 3: Quiet Bio-inspired Propulsion System Designed By: Henry Bryant Printed On: March 12th, 2026"

Commit message: control board ordered
Parts:
- added P1: SolderBridge_GND, bio-robot:SolderBridge_GND, F.Cu at (147.5, 112.5)
- added P2: SolderBridge_GND, bio-robot:SolderBridge_GND, F.Cu at (151.0, 112.5)
- added P3: SolderBridge_GND, bio-robot:SolderBridge_GND, F.Cu at (154.5, 112.5)
- added P4: SolderBridge_GND, bio-robot:SolderBridge_GND, F.Cu at (158.0, 112.5)
- added P5: SolderBridge_GND, bio-robot:SolderBridge_GND, F.Cu at (161.5, 112.5)
- M1, M2, M3, M4, M5, M6, M7, M8: footprint bio-robot:PinSocket_1x03_P2.54mm_Vertical -> bio-robot:PinHeader_1x03_P2.54mm_Vertical
Routing:
- net GNDPWR: vias 6 -> 22
- net GND: vias 4 -> 20
- added copper zone on B.Cu, net GND
- added copper zone on F.Cu, net GND
- added copper zone on B.Cu, net GNDPWR
- added copper zone on F.Cu, net GNDPWR
Other:
- board text added: "+"
- board text added: "-"
- board text added: "1"
- board text added: "10"
- board text added: "11"
- board text added: "12"
- board text added: "13"
- board text added: "14"
- board text added: "15"
- board text added: "16"
- board text added: "17"
- board text added: "18"
- board text added: "2"
- board text added: "21"
- board text added: "3"
- board text added: "3.3V"
- board text added: "39"
- board text added: "4"
- board text added: "40"
- board text added: "41"
- board text added: "42"
- board text added: "45"
- board text added: "47"
- board text added: "48"
- board text added: "5"
- board text added: "6"
- board text added: "7"
- board text added: "8"
- board text added: "9"
- board text added: "AD0"
- board text added: "D+"
- board text added: "D-"
- board text added: "FLAG"
- board text added: "IF ISOLATORS DNP: BRIDGE GND"
- board text added: "INT"
- board text added: "PWM"
- board text added: "SCL"
- board text added: "SDA"
- board text added: "XCL"
- board text added: "XDA"
