File: servo-board/servo-board.kicad_sch (KiCad schematic)
At the start: 7 parts, among them M1 Motor_Servo, M2 Motor_Servo, M3 Motor_Servo, M4 Motor_Servo, M5 Motor_Servo, M6 Motor_Servo, U1 ESP32-S3-DEVKITC-1-N8R8

Commit message: board
Parts:
- added H1, H2, H3, H4: MountingHoleM3, MountingHole:MountingHole_3.2mm_M3_DIN965_Pad, symbol bio-robot:MountingHoleM3
- added J1, J2: Screw_Terminal_01x02, TerminalBlock:TerminalBlock_MaiXu_MX126-5.0-02P_1x02_P5.00mm, symbol bio-robot:Screw_Terminal_01x02
- added J3: Conn_02x10_Counter_Clockwise, Connector_PinSocket_2.54mm:PinSocket_2x10_P2.54mm_Vertical, symbol bio-robot:Conn_02x10
- added M7, M8: Motor_Servo, Connector_PinSocket_2.54mm:PinSocket_1x03_P2.54mm_Vertical, symbol bio-robot:Motor_Servo
- added U2: GY-521_MPU-6050, bio-robot:MODULE_OC09600, symbol bio-robot:GY-521_MPU-6050
- U1: footprint ESP32-S3-DEVKITC-1-N8R8:ESP32-S3-DEVKITC-1-N8R8 -> bio-robot:ESP32-S3-DEVKITC-1-N8R8
Connections:
- net +3V3: now reaches U1.J1_1 (3V3)
- net +3V3: now also U1.J1_2 (3V3.), J3.1 (Pin_1), U2.VCC
- net GPIO17: now reaches U1.J1_10 (GPIO17)
- net GPIO17: now also J3.13 (Pin_13)
- net GPIO18: now reaches U1.J1_11 (GPIO18)
- net GPIO18: now also J3.15 (Pin_15)
- net SDA: now reaches U1.J1_12 (GPIO8)
- net SDA: now also U2.SDA
- net GPIO3: now reaches U1.J1_13 (GPIO3)
- net GPIO3: now also J3.5 (Pin_5)
- net GPIO46: now reaches U1.J1_14 (GPIO46)
- net GPIO46: now also J3.7 (Pin_7)
- net SCL: now reaches U1.J1_15 (GPIO9)
- net SCL: now also U2.SCL
- net INT: now reaches U1.J1_16 (GPIO10)
- net INT: now also U2.INT
- net PWM_M5: now reaches U1.J1_17 (GPIO11)
- net PWM_M5: now also M5.1 (PWM)
- net PWM_M6: now reaches U1.J1_18 (GPIO12)
- net PWM_M6: now also M6.1 (PWM)
- net PWM_M7: now reaches U1.J1_19 (GPIO13)
- net PWM_M7: now also M7.1 (PWM)
- net PWM_M8: now reaches U1.J1_20 (GPIO14)
- net PWM_M8: now also M8.1 (PWM)
- net +5V: now reaches U1.J1_21 (5V0)
- net +5V: now also J1.1 (Pin_1)
- net GND: now reaches U1.J1_22 (GND3)
- net GND: now also U1.J3_1 (GND), U1.J3_21 (GND1), U1.J3_22 (GND2), J1.2 (Pin_2), J3.3 (Pin_3), U2.GND
- net PWM_M1: now reaches U1.J1_4 (GPIO4)
- net PWM_M1: now also M1.1 (PWM)
- net PWM_M2: now reaches U1.J1_5 (GPIO5)
- net PWM_M2: now also M2.1 (PWM)
- net PWM_M3: now reaches U1.J1_6 (GPIO6)
- net PWM_M3: now also M3.1 (PWM)
- net PWM_M4: now reaches U1.J1_7 (GPIO7)
- net PWM_M4: now also M4.1 (PWM)
- net GPIO15: now reaches U1.J1_8 (GPIO15)
- net GPIO15: now also J3.9 (Pin_9)
- net GPIO16: now reaches U1.J1_9 (GPIO16)
- net GPIO16: now also J3.11 (Pin_11)
- net GPI45: now reaches U1.J3_15 (GPIO45)
- net GPI45: now also J3.14 (Pin_14)
- net GPI48: now reaches U1.J3_16 (GPIO48)
- net GPI48: now also J3.16 (Pin_16)
- net GPI47: now reaches U1.J3_17 (GPIO47)
- net GPI47: now also J3.18 (Pin_18)
- net GPIO21: now reaches U1.J3_18 (GPIO21)
- net GPIO21: now also J3.20 (Pin_20)
- net GPIO20_USB_D+: now reaches U1.J3_19 (USB_D+/GPIO20)
- net GPIO20_USB_D+: now also J3.17 (Pin_17)
- net GPIO19_USB_D-: now reaches U1.J3_20 (USB_D-/GPIO19)
- net GPIO19_USB_D-: now also J3.19 (Pin_19)
- net GPIO1: now reaches U1.J3_4 (GPIO1)
- net GPIO1: now also J3.2 (Pin_2)
- net GPIO2: now reaches U1.J3_5 (GPIO2)
- net GPIO2: now also J3.4 (Pin_4)
- net MTMS_GPIO42: now reaches U1.J3_6 (MTMS/GPIO42)
- net MTMS_GPIO42: now also J3.6 (Pin_6)
- net MTDI_GPIO41: now reaches U1.J3_7 (MTDI/GPIO41)
- net MTDI_GPIO41: now also J3.8 (Pin_8)
- net MTDO_GPIO40: now reaches U1.J3_8 (MTDO/GPIO40)
- net MTDO_GPIO40: now also J3.10 (Pin_10)
- net MTCK_GPIO39: now reaches U1.J3_9 (MTCK/GPIO39)
- net MTCK_GPIO39: now also J3.12 (Pin_12)
- net +6.8V: now reaches M3.2 (+)
- net +6.8V: now also M1.2 (+), M2.2 (+), M4.2 (+), M5.2 (+), M6.2 (+), J2.1 (Pin_1), M7.2 (+), M8.2 (+)
- net GNDPWR: now reaches M3.3 (-)
- net GNDPWR: now also M1.3 (-), M2.3 (-), M4.3 (-), M5.3 (-), M6.3 (-), J2.2 (Pin_2), M7.3 (-), M8.3 (-)
- no-connect marks 0 -> 11
Other:
- moved on the sheet: M2, M3, M4, M5, M6, U1

Commit message: board done
Parts:
- removed M1, M2, M3, M4, M5, M6, M7, M8: Motor_Servo, Connector_PinSocket_2.54mm:PinSocket_1x03_P2.54mm_Vertical, symbol bio-robot:Motor_Servo
- H1, H2, H3, H4: footprint MountingHole:MountingHole_3.2mm_M3_DIN965_Pad -> bio-robot:MountingHole_3.2mm_M3_DIN965_Pad
- J1, J2: footprint TerminalBlock:TerminalBlock_MaiXu_MX126-5.0-02P_1x02_P5.00mm -> bio-robot:TerminalBlock_MaiXu_MX126-5.0-02P_1x02_P5.00mm
- J3: footprint Connector_PinSocket_2.54mm:PinSocket_2x10_P2.54mm_Vertical -> bio-robot:PinSocket_2x10_P2.54mm_Vertical
Connections:
- net INT: now also U1.J1_13 (GPIO3); no longer U1.J1_16 (GPIO10)
- net PWM_M5: now also U1.J1_19 (GPIO13); no longer U1.J1_17 (GPIO11)
- net PWM_M7: now also U1.J1_17 (GPIO11); no longer U1.J1_19 (GPIO13)
- net PWM_M8: now also U1.J1_16 (GPIO10); no longer U1.J1_20 (GPIO14)
- net GPIO19_USB_D- renamed USB_D-
- net GPIO20_USB_D+ renamed USB_D+
- net GPIO3 renamed GPIO14
- net GPIO14: now also U1.J1_20 (GPIO14); no longer U1.J1_13 (GPIO3)
- net GPIO46 renamed FLAG
Other:
- added sheet servos (servos.kicad_sch)

Commit message: changes
Other:
- note added: "ESP32S3 Dev Module"
- note added: "IMU Header (MPU 6050)"
- note added: "M3 Mounting Holes"
- note added: "Power Input + GPIO Header (Extra pins)"
- note added: "Servos"
- moved on the sheet: H1, H2, H3, H4, J1, J2, J3, U1, U2
