File: motherboard-esp32/dc-dc.kicad_sch (KiCad schematic)
At the start: 27 parts, among them J2 Screw_Terminal_01x02, J5 Screw_Terminal_01x02, J6 Screw_Terminal_01x02, P1 1.8mm_16AWG, P2 1.8mm_16AWG, P3 1.8mm_16AWG, P4 1.8mm_16AWG, U2 LMR51450SDRRR

Commit message: ordered
Parts:
- removed H10, H9: MountingHoleM3, bio-robot:MountingHole_3.2mm_M3_DIN965_Pad, symbol bio-robot:MountingHoleM3
Changed lines of the file:
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@@
-	)
-	(symbol
-		(lib_id "bio-robot:MountingHoleM3")
-		(at 90.17 121.92 0)
-		(unit 1)
-		(body_style 1)
-		(exclude_from_sim no)
-		(in_bom no)
-		(on_board yes)
-		(in_pos_files yes)
-		(dnp no)
-		(fields_autoplaced yes)
-		(property "Reference" "H9"
-			(at 92.71 120.6499 0)
-			(show_name no)
-			(do_not_autoplace no)
-			(effects
-				(font
-					(size 1.27 1.27)
-				)
-				(justify left)
-			)
-		)
-		(property "Value" "MountingHoleM3"
-			(at 92.71 123.1899 0)
-			(show_name no)
-			(do_not_autoplace no)
-			(effects
-				(font
-					(size 1.27 1.27)
-				)
-				(justify left)
-			)
-		)
-		(property "Footprint" "bio-robot:MountingHole_3.2mm_M3_DIN965_Pad"
-			(at 90.17 121.92 0)
-			(hide yes)
-			(show_name no)
-			(do_not_autoplace no)
-			(effects
-				(font
-					(size 1.27 1.27)
-				)
-			)
-		)
-		(property "Datasheet" ""
-			(at 90.17 121.92 0)
-			(hide yes)
-			(show_name no)
-			(do_not_autoplace no)
-			(effects
-				(font
-					(size 1.27 1.27)
-				)
-			)
-		)
-		(property "Description" "Mounting Hole without connection"
-			(at 90.17 121.92 0)
-			(hide yes)
-			(show_name no)
-			(do_not_autoplace no)
-			(effects
-				(font
-					(size 1.27 1.27)
-				)
-			)
-		)
-		(instances
-			(project "motherboard-esp32"
-				(path "/d5fb8fba-70d9-4abd-aa21-c96ccdcfa753/78ac5bff-7e06-43c5-8f16-db859d5291bc"
-					(reference "H9")
-					(unit 1)
-				)
-			)
-		)
 	)
 	(symbol
@@
 					(unit 1)
 				)
-			)
-		)
-	)
-	(symbol
-		(lib_id "bio-robot:MountingHoleM3")
-		(at 90.17 130.81 0)
-		(unit 1)
-		(body_style 1)
-		(exclude_from_sim no)
-		(in_bom no)
-		(on_board yes)
-		(in_pos_files yes)
-		(dnp no)
-		(fields_autoplaced yes)
-		(property "Reference" "H10"
-			(at 92.71 129.5399 0)
-			(show_name no)
-			(do_not_autoplace no)
-			(effects
-				(font
-					(size 1.27 1.27)
-				)
-				(justify left)
-			)
-		)
-		(property "Value" "MountingHoleM3"
-			(at 92.71 132.0799 0)
-			(show_name no)
-			(do_not_autoplace no)
-			(effects
-				(font
-					(size 1.27 1.27)
-				)
-				(justify left)
-			)
-		)
-		(property "Footprint" "bio-robot:MountingHole_3.2mm_M3_DIN965_Pad"
-			(at 90.17 130.81 0)
-			(hide yes)
-			(show_name no)
-			(do_not_autoplace no)
-			(effects
-				(font
-					(size 1.27 1.27)
-				)
-			)
-		)
-		(property "Datasheet" ""
-			(at 90.17 130.81 0)
-			(hide yes)
-			(show_name no)
-			(do_not_autoplace no)
-			(effects
-				(font
-					(size 1.27 1.27)
-				)
-			)
-		)
-		(property "Description" "Mounting Hole without connection"
-			(at 90.17 130.81 0)
-			(hide yes)
-			(show_name no)
-			(do_not_autoplace no)
-			(effects
-				(font
-					(size 1.27 1.27)
-				)
-			)
-		)
-		(instances
-			(project "motherboard-esp32"
-				(path "/d5fb8fba-70d9-4abd-aa21-c96ccdcfa753/78ac5bff-7e06-43c5-8f16-db859d5291bc"
-					(reference "H10")
-					(unit 1)
-				)
