File: motherboard-esp32/power-input.kicad_sch (KiCad schematic)
At the start: 26 parts, among them J3 JST_2P_XH, J4 JST_2P_XH, J7 XT60, Q1 DOD4185, Q2 DOD4185, Q3 DOD4185, Q4 DOD4185, Q6 TN2130K1-G

Commit message: changes
Parts:
- D6: value LED_blue -> LED_white
Other:
- moved on the sheet: D3, R7
Changed lines of the file:
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@@
 	(wire
 		(pts
-			(xy 222.25 36.83) (xy 222.25 39.37)
+			(xy 185.42 119.38) (xy 185.42 123.19)
 		)
 		(stroke
@@
 	(wire
 		(pts
-			(xy 222.25 58.42) (xy 222.25 62.23)
+			(xy 185.42 142.24) (xy 185.42 146.05)
 		)
 		(stroke
@@
 	(wire
 		(pts
-			(xy 34.29 143.51) (xy 34.29 110.49)
+			(xy 34.29 147.32) (xy 34.29 110.49)
 		)
 		(stroke
@@
 	(wire
 		(pts
-			(xy 101.6 142.24) (xy 111.76 142.24)
+			(xy 97.79 142.24) (xy 111.76 142.24)
 		)
 		(stroke
@@
 	(wire
 		(pts
-			(xy 101.6 142.24) (xy 101.6 167.64)
+			(xy 97.79 142.24) (xy 97.79 147.32)
 		)
 		(stroke
@@
 	(wire
 		(pts
-			(xy 222.25 46.99) (xy 222.25 50.8)
+			(xy 185.42 130.81) (xy 185.42 134.62)
 		)
 		(stroke
@@
 	)
 	(label "LED_5V"
-		(at 222.25 49.53 0)
+		(at 185.42 133.35 0)
 		(effects
 			(font
@@
 			)
 		)
-		(property "Value" "LED_blue"
+		(property "Value" "LED_white"
 			(at 234.95 142.3378 90)
 			(show_name no)
@@
 	(symbol
 		(lib_id "bio-robot:LED_green")
-		(at 222.25 54.61 90)
+		(at 185.42 138.43 90)
 		(unit 1)
 		(body_style 1)
@@
 		(fields_autoplaced yes)
 		(property "Reference" "D3"
-			(at 226.06 54.9274 90)
+			(at 189.23 138.7474 90)
 			(show_name no)
 			(do_not_autoplace no)
@@
 		)
 		(property "Value" "LED_green"
-			(at 226.06 57.4674 90)
+			(at 189.23 141.2874 90)
 			(show_name no)
 			(do_not_autoplace no)
@@
 		)
 		(property "Footprint" "bio-robot:LED_0805_2012Metric"
-			(at 229.87 54.61 0)
+			(at 193.04 138.43 0)
 			(hide yes)
 			(show_name no)
@@
 		)
 		(property "Datasheet" ""
-			(at 222.25 54.61 0)
+			(at 185.42 138.43 0)
 			(hide yes)
 			(show_name no)
@@
 		)
 		(property "Description" "Light emitting diode"
-			(at 222.25 54.61 0)
+			(at 185.42 138.43 0)
 			(hide yes)
 			(show_name no)
@@
 		)
 		(property "MPN" "KT-0805G"
-			(at 229.87 54.61 0)
+			(at 193.04 138.43 0)
 			(hide yes)
 			(show_name no)
@@
 		)
 		(property "Manufacturer" "Hubei KENTO Elec"
-			(at 228.6 54.61 0)
+			(at 191.77 138.43 0)
 			(hide yes)
 			(show_name no)
@@
 		)
 		(property "Price" "0.0127"
-			(at 228.6 54.61 0)
+			(at 191.77 138.43 0)
 			(hide yes)
 			(show_name no)
@@
 		)
 		(property "JLC" "0805"
-			(at 228.6 53.34 0)
+			(at 191.77 137.16 0)
 			(hide yes)
 			(show_name no)
@@
 		)
 		(property "LCSC" "C2297"
-			(at 229.87 54.61 0)
+			(at 193.04 138.43 0)
 			(hide yes)
 			(show_name no)
@@
 		)
 		(property "JLC Extended" "no"
-			(at 222.25 54.61 0)
+			(at 185.42 138.43 0)
 			(hide yes)
 			(show_name no)
@@
 	(symbol
 		(lib_id "power:GND")
-		(at 34.29 143.51 0)
+		(at 34.29 147.32 0)
 		(unit 1)
 		(body_style 1)
@@
 		(dnp no)
 		(property "Reference" "#PWR017"
-			(at 34.29 149.86 0)
+			(at 34.29 153.67 0)
 			(hide yes)
 			(show_name no)
@@
 		)
 		(property "Value" "GND"
-			(at 34.29 147.32 0)
+			(at 34.29 151.13 0)
 			(show_name no)
 			(do_not_autoplace no)
@@
 		)
 		(property "Footprint" ""
-			(at 34.29 143.51 0)
+			(at 34.29 147.32 0)
 			(hide yes)
 			(show_name no)
@@
 		)
 		(property "Datasheet" ""
-			(at 34.29 143.51 0)
+			(at 34.29 147.32 0)
 			(hide yes)
 			(show_name no)
@@
 		)
 		(property "Description" "Power symbol creates a global label with name \"GND\" , ground"
-			(at 34.29 143.51 0)
+			(at 34.29 147.32 0)
 			(hide yes)
 			(show_name no)
@@
 	(symbol
 		(lib_id "power:GND")
-		(at 101.6 167.64 0)
+		(at 97.79 147.32 0)
 		(unit 1)
 		(body_style 1)
@@
 		(dnp no)
 		(property "Reference" "#PWR018"
-			(at 101.6 173.99 0)
+			(at 97.79 153.67 0)
 			(hide yes)
 			(show_name no)
@@
 		)
 		(property "Value" "GND"
-			(at 101.6 171.45 0)
+			(at 97.79 151.13 0)
 			(show_name no)
 			(do_not_autoplace no)
@@
 		)
 		(property "Footprint" ""
-			(at 101.6 167.64 0)
+			(at 97.79 147.32 0)
 			(hide yes)
 			(show_name no)
@@
 		)
 		(property "Datasheet" ""
-			(at 101.6 167.64 0)
+			(at 97.79 147.32 0)
 			(hide yes)
 			(show_name no)
@@
 		)
 		(property "Description" "Power symbol creates a global label with name \"GND\" , ground"
-			(at 101.6 167.64 0)
+			(at 97.79 147.32 0)
 			(hide yes)
 			(show_name no)
@@
 	(symbol
 		(lib_id "power:GND")
-		(at 222.25 62.23 0)
+		(at 185.42 146.05 0)
 		(unit 1)
 		(body_style 1)
@@
 		(dnp no)
 		(property "Reference" "#PWR050"
-			(at 222.25 68.58 0)
+			(at 185.42 152.4 0)
 			(hide yes)
 			(show_name no)
@@
 		)
 		(property "Value" "GND"
-			(at 223.52 66.294 0)
+			(at 186.69 150.114 0)
 			(show_name no)
 			(do_not_autoplace no)
@@
 		)
 		(property "Footprint" ""
-			(at 222.25 62.23 0)
+			(at 185.42 146.05 0)
 			(hide yes)
 			(show_name no)
@@
 		)
 		(property "Datasheet" ""
-			(at 222.25 62.23 0)
+			(at 185.42 146.05 0)
 			(hide yes)
 			(show_name no)
@@
 		)
 		(property "Description" "Power symbol creates a global label with name \"GND\" , ground"
-			(at 222.25 62.23 0)
+			(at 185.42 146.05 0)
 			(hide yes)
 			(show_name no)
@@
 	(symbol
 		(lib_id "bio-robot:R_3.3k")
-		(at 222.25 43.18 0)
+		(at 185.42 127 0)
 		(unit 1)
 		(body_style 1)
@@
 		(fields_autoplaced yes)
 		(property "Reference" "R7"
-			(at 224.79 41.9099 0)
+			(at 187.96 125.7299 0)
 			(show_name no)
 			(do_not_autoplace no)
@@
 		)
 		(property "Value" "3.3k"
-			(at 224.79 44.4499 0)
+			(at 187.96 128.2699 0)
 			(show_name no)
 			(do_not_autoplace no)
@@
 		)
 		(property "Footprint" "bio-robot:R_0603_1608Metric"
-			(at 220.472 43.18 90)
+			(at 183.642 127 90)
 			(hide yes)
 			(show_name no)
@@
 		)
 		(property "Datasheet" ""
-			(at 222.25 43.18 0)
+			(at 185.42 127 0)
 			(hide yes)
 			(show_name no)
@@
 		)
 		(property "Description" "Resistor"
-			(at 222.25 43.18 0)
+			(at 185.42 127 0)
 			(hide yes)
 			(show_name no)
@@
 		)
 		(property "MPN" "0603WAF3301T5E"
-			(at 222.25 43.18 0)
+			(at 185.42 127 0)
 			(hide yes)
 			(show_name no)
@@
 		)
 		(property "Manufacturer" "UNI-ROYAL(Uniroyal Elec)"
-			(at 222.25 43.18 0)
+			(at 185.42 127 0)
 			(hide yes)
 			(show_name no)
@@
 		)
 		(property "Price" "0.0009"
-			(at 222.25 43.18 0)
+			(at 185.42 127 0)
 			(hide yes)
 			(show_name no)
@@
 		)
 		(property "JLC" "0603"
-			(at 222.25 43.18 0)
+			(at 185.42 127 0)
 			(hide yes)
 			(show_name no)
@@
 		)
 		(property "LCSC" "C22978"
-			(at 222.25 43.18 0)
+			(at 185.42 127 0)
 			(hide yes)
 			(show_name no)
@@
 		)
 		(property "JLC Extended" "no"
-			(at 222.25 43.18 0)
+			(at 185.42 127 0)
 			(hide yes)
 			(show_name no)
@@
 	(symbol
 		(lib_id "power:+5V")
-		(at 222.25 36.83 0)
+		(at 185.42 119.38 0)
 		(unit 1)
 		(body_style 1)
@@
 		(dnp no)
 		(property "Reference" "#PWR049"
-			(at 222.25 40.64 0)
+			(at 185.42 123.19 0)
 			(hide yes)
 			(show_name no)
@@
 		)
 		(property "Value" "+5V"
-			(at 222.25 33.274 0)
+			(at 185.42 115.824 0)
 			(show_name no)
 			(do_not_autoplace no)
@@
 		)
 		(property "Footprint" ""
-			(at 222.25 36.83 0)
+			(at 185.42 119.38 0)
 			(hide yes)
 			(show_name no)
@@
 		)
 		(property "Datasheet" ""
-			(at 222.25 36.83 0)
+			(at 185.42 119.38 0)
 			(hide yes)
 			(show_name no)
@@
 		)
 		(property "Description" "Power symbol creates a global label with name \"+5V\""
-			(at 222.25 36.83 0)
+			(at 185.42 119.38 0)
 			(hide yes)
 			(show_name no)

Commit message: zener notes
Other:
- note added: "- these mosfets turn on at -5 to -5.5V fully, not -3V as specced. Just keep that in mind."
- note added: "need the zener to clamp the voltage at minimum voltage 6.4V - 5.5 = 0.9V (3.6V Zener doesnt work here , and is likely unfeasible unless a lower Vth mosfet is chosen)"
- note added: "need the zener to clamp the voltage at minimum voltage 9.6V - 5.5 = 4.1V (4.7V Zener doesnt work here at voltages < 10.3V)"
- moved on the sheet: D3, R7
Changed lines of the file:
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@@
 		)
 	)
+	(text "need the zener to clamp the voltage at minimum voltage\n9.6V - 5.5 = 4.1V (4.7V Zener doesnt work here at voltages < 10.3V)"
+		(exclude_from_sim no)
+		(at 175.514 38.608 0)
+		(effects
+			(font
+				(size 1.27 1.27)
+			)
+		)
+	)
+	(text "- these mosfets turn on at -5 to -5.5V fully, not -3V as specced. Just keep that in mind. "
+		(exclude_from_sim no)
+		(at 162.56 110.49 0)
+		(effects
+			(font
+				(size 1.27 1.27)
+			)
+		)
+	)
+	(text "need the zener to clamp the voltage at minimum voltage\n6.4V - 5.5 = 0.9V (3.6V Zener doesnt work here\n, and is likely unfeasible unless a lower Vth mosfet is chosen)"
+		(exclude_from_sim no)
+		(at 148.844 116.078 0)
+		(effects
+			(font
+				(size 1.27 1.27)
+			)
+		)
+	)
+	(text "- these mosfets turn on at -5 to -5.5V fully, not -3V as specced. Just keep that in mind. "
+		(exclude_from_sim no)
+		(at 189.738 33.528 0)
+		(effects
+			(font
+				(size 1.27 1.27)
+			)
+		)
+	)
 	(junction
 		(at 110.49 73.66)
@@
 	(wire
 		(pts
-			(xy 185.42 119.38) (xy 185.42 123.19)
+			(xy 228.6 44.45) (xy 228.6 48.26)
 		)
 		(stroke
@@
 	(wire
 		(pts
-			(xy 185.42 142.24) (xy 185.42 146.05)
+			(xy 228.6 67.31) (xy 228.6 71.12)
 		)
 		(stroke
@@
 	(wire
 		(pts
-			(xy 185.42 130.81) (xy 185.42 134.62)
+			(xy 228.6 55.88) (xy 228.6 59.69)
 		)
 		(stroke
@@
 	)
 	(label "LED_5V"
-		(at 185.42 133.35 0)
+		(at 228.6 58.42 0)
 		(effects
 			(font
@@
 	(symbol
 		(lib_id "bio-robot:LED_green")
-		(at 185.42 138.43 90)
+		(at 228.6 63.5 90)
 		(unit 1)
 		(body_style 1)
@@
 		(fields_autoplaced yes)
 		(property "Reference" "D3"
-			(at 189.23 138.7474 90)
+			(at 232.41 63.8174 90)
 			(show_name no)
 			(do_not_autoplace no)
@@
 		)
 		(property "Value" "LED_green"
-			(at 189.23 141.2874 90)
+			(at 232.41 66.3574 90)
 			(show_name no)
 			(do_not_autoplace no)
@@
 		)
 		(property "Footprint" "bio-robot:LED_0805_2012Metric"
-			(at 193.04 138.43 0)
+			(at 236.22 63.5 0)
 			(hide yes)
 			(show_name no)
@@
 		)
 		(property "Datasheet" ""
-			(at 185.42 138.43 0)
+			(at 228.6 63.5 0)
 			(hide yes)
 			(show_name no)
@@
 		)
 		(property "Description" "Light emitting diode"
-			(at 185.42 138.43 0)
+			(at 228.6 63.5 0)
 			(hide yes)
 			(show_name no)
@@
 		)
 		(property "MPN" "KT-0805G"
-			(at 193.04 138.43 0)
+			(at 236.22 63.5 0)
 			(hide yes)
 			(show_name no)
@@
 		)
 		(property "Manufacturer" "Hubei KENTO Elec"
-			(at 191.77 138.43 0)
+			(at 234.95 63.5 0)
 			(hide yes)
 			(show_name no)
@@
 		)
 		(property "Price" "0.0127"
-			(at 191.77 138.43 0)
+			(at 234.95 63.5 0)
 			(hide yes)
 			(show_name no)
@@
 		)
 		(property "JLC" "0805"
-			(at 191.77 137.16 0)
+			(at 234.95 62.23 0)
 			(hide yes)
 			(show_name no)
@@
 		)
 		(property "LCSC" "C2297"
-			(at 193.04 138.43 0)
+			(at 236.22 63.5 0)
 			(hide yes)
 			(show_name no)
@@
 		)
 		(property "JLC Extended" "no"
-			(at 185.42 138.43 0)
+			(at 228.6 63.5 0)
 			(hide yes)
 			(show_name no)
@@
 	(symbol
 		(lib_id "power:GND")
-		(at 185.42 146.05 0)
+		(at 228.6 71.12 0)
 		(unit 1)
 		(body_style 1)
@@
 		(dnp no)
 		(property "Reference" "#PWR050"
-			(at 185.42 152.4 0)
+			(at 228.6 77.47 0)
 			(hide yes)
 			(show_name no)
@@
 		)
 		(property "Value" "GND"
-			(at 186.69 150.114 0)
+			(at 229.87 75.184 0)
 			(show_name no)
 			(do_not_autoplace no)
@@
 		)
 		(property "Footprint" ""
-			(at 185.42 146.05 0)
+			(at 228.6 71.12 0)
 			(hide yes)
 			(show_name no)
@@
 		)
 		(property "Datasheet" ""
-			(at 185.42 146.05 0)
+			(at 228.6 71.12 0)
 			(hide yes)
 			(show_name no)
@@
 		)
 		(property "Description" "Power symbol creates a global label with name \"GND\" , ground"
-			(at 185.42 146.05 0)
+			(at 228.6 71.12 0)
 			(hide yes)
 			(show_name no)
@@
 	(symbol
 		(lib_id "bio-robot:R_3.3k")
-		(at 185.42 127 0)
+		(at 228.6 52.07 0)
 		(unit 1)
 		(body_style 1)
@@
 		(fields_autoplaced yes)
 		(property "Reference" "R7"
-			(at 187.96 125.7299 0)
+			(at 231.14 50.7999 0)
 			(show_name no)
 			(do_not_autoplace no)
@@
 		)
 		(property "Value" "3.3k"
-			(at 187.96 128.2699 0)
+			(at 231.14 53.3399 0)
 			(show_name no)
 			(do_not_autoplace no)
@@
 		)
 		(property "Footprint" "bio-robot:R_0603_1608Metric"
-			(at 183.642 127 90)
+			(at 226.822 52.07 90)
 			(hide yes)
 			(show_name no)
@@
 		)
 		(property "Datasheet" ""
-			(at 185.42 127 0)
+			(at 228.6 52.07 0)
 			(hide yes)
 			(show_name no)
@@
 		)
 		(property "Description" "Resistor"
-			(at 185.42 127 0)
+			(at 228.6 52.07 0)
 			(hide yes)
 			(show_name no)
@@
 		)
 		(property "MPN" "0603WAF3301T5E"
-			(at 185.42 127 0)
+			(at 228.6 52.07 0)
 			(hide yes)
 			(show_name no)
@@
 		)
 		(property "Manufacturer" "UNI-ROYAL(Uniroyal Elec)"
-			(at 185.42 127 0)
+			(at 228.6 52.07 0)
 			(hide yes)
 			(show_name no)
@@
 		)
 		(property "Price" "0.0009"
-			(at 185.42 127 0)
+			(at 228.6 52.07 0)
 			(hide yes)
 			(show_name no)
@@
 		)
 		(property "JLC" "0603"
-			(at 185.42 127 0)
+			(at 228.6 52.07 0)
 			(hide yes)
 			(show_name no)
@@
 		)
 		(property "LCSC" "C22978"
-			(at 185.42 127 0)
+			(at 228.6 52.07 0)
 			(hide yes)
 			(show_name no)
@@
 		)
 		(property "JLC Extended" "no"
-			(at 185.42 127 0)
+			(at 228.6 52.07 0)
 			(hide yes)
 			(show_name no)
@@
 	(symbol
 		(lib_id "power:+5V")
-		(at 185.42 119.38 0)
+		(at 228.6 44.45 0)
 		(unit 1)
 		(body_style 1)
@@
 		(dnp no)
 		(property "Reference" "#PWR049"
-			(at 185.42 123.19 0)
+			(at 228.6 48.26 0)
 			(hide yes)
 			(show_name no)
@@
 		)
 		(property "Value" "+5V"
-			(at 185.42 115.824 0)
+			(at 228.6 40.894 0)
 			(show_name no)
 			(do_not_autoplace no)
@@
 		)
 		(property "Footprint" ""
-			(at 185.42 119.38 0)
+			(at 228.6 44.45 0)
 			(hide yes)
 			(show_name no)
@@
 		)
 		(property "Datasheet" ""
-			(at 185.42 119.38 0)
+			(at 228.6 44.45 0)
 			(hide yes)
 			(show_name no)
@@
 		)
 		(property "Description" "Power symbol creates a global label with name \"+5V\""
-			(at 185.42 119.38 0)
+			(at 228.6 44.45 0)
 			(hide yes)
 			(show_name no)
