File: battery-motherboard/battery-motherboard.kicad_pcb (KiCad board)
At the start: 4 copper layers, 123.8 x 77 mm, 58 parts, among them J2 Screw_Terminal_01x02, J3 JST_2P_XH, J4 JST_2P_XH, J5 Screw_Terminal_01x02, J6 Screw_Terminal_01x02, J7 XT60, P1 1.8mm_16AWG, P2 1.8mm_16AWG, P3 1.8mm_16AWG, P4 1.8mm_16AWG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

Commit message: changes
Other:
- board text added: "NEED TO FIX THE CURRENT BOTTLENECK FOR 12V TERMINAL BLOCK"
- board text added: "This board has two battery inputs. - 5V Rail: 2-Cell 18650 Protected (Li-Ion). Buck to 5V 5A. - 12V Rail: 3-Cell Custom Battery Pack using XT60. Buck to 6.8V, 10A."
- board text removed: "This board has two battery inputs. - 5V Rail: 2-Cell 18650 Protected (Li-Ion). Buck to 5V 3A. - 12V Rail: 3-Cell Custom Battery Pack using XT60. Buck to 6.8V, 10A."
Changed lines of the file:
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@@
 		(layer "Edge.Cuts")
 	)
-	(gr_text "This board has two battery inputs.\n- 5V Rail: 2-Cell 18650 Protected (Li-Ion). \n	Buck to 5V 3A.\n- 12V Rail: 3-Cell Custom Battery Pack using XT60. \n	Buck to 6.8V, 10A."
+	(gr_text "This board has two battery inputs.\n- 5V Rail: 2-Cell 18650 Protected (Li-Ion). \n	Buck to 5V 5A.\n- 12V Rail: 3-Cell Custom Battery Pack using XT60. \n	Buck to 6.8V, 10A."
 		(at 70.7 91.25 0)
 		(layer "F.SilkS")
 		(effects
+			(font
+				(size 1 1)
+				(thickness 0.15)
+			)
+			(justify left bottom)
+		)
+	)
+	(gr_text "NEED TO FIX THE CURRENT BOTTLENECK \nFOR 12V TERMINAL BLOCK\n"
+		(at 175.75 81 0)
+		(layer "F.SilkS")
+		(effects
