File: battery-motherboard/dc-dc.kicad_sch (KiCad schematic)
At the start: 25 parts, among them J2 Screw_Terminal_01x02, J5 Screw_Terminal_01x02, J6 Screw_Terminal_01x02, P1 1.8mm_16AWG, P2 1.8mm_16AWG, P3 1.8mm_16AWG, P4 1.8mm_16AWG, U2 LMR51450SDRRR

Commit message: naming
Other:
- note added: "for Logic supply or Raspberry Pi boards (3-5A needed)"
- note removed: "for Raspberry Pi boards (for other projects)"
- moved on the sheet: C1, C2, C4, H5, H6, H7, H8, L1, R15, R5, R6
