File: battery-motherboard/power-input.kicad_sch (KiCad schematic)
At the start: 26 parts, among them J3 JST_2P_XH, J4 JST_2P_XH, J7 XT60, Q1 DOD4185, Q2 DOD4185, Q3 DOD4185, Q4 DOD4185, Q6 TN2130K1-G

Commit message: naming
Other:
- note added: "Final Resistor Values for approx equal intensity: 5V: (5V-2.29)/6.8k = 0.4mA (1/2 brightness) 6.8V: (6.8V-2.57V)/4.7k = 0.9mA (1/2 brightness) VCC: (9.6 to 12.6V-1.79V)/10k = 0.8mA to 1.1mA"
- note added: "LED drops 1.79V on a multimeter 9.6-12.6V: worst case = 12.6V (12.6V-1.79V)/34k = 0.32mA (this is dim). We want ~1mA (12.6V-1.79V)/1mA = 10.8k"
- note added: "LED drops 2.57V across it. (6.8V-2.57V)/2k = 2.1mA (this is fairly bright) reduce to 1mA (6.8V-2.57V)/1mA = 4.3k"
- note added: "Led drops 2.29V on multimeter (5V-2.29V)/3.3k = 0.82 ( bright). Could reduce. Perhaps 0.5mA is ideal? (5V-2.29V)/0.5mA = 5.4k; raise to 6.8k"
- moved on the sheet: B1
